File: KiCAD/K40-LED_PCB/K40-LED_PCB.kicad_pcb (KiCad board)
At the start: 2 copper layers, 106.9 x 56.9 mm, 11 parts, among them J2 54-00166, M3 MountingHole_3.2mm_M3, U1 LDD_350HS

Commit message: Update
Other:
- board text added: "NHB [2024]"
- board text added: "locked"
- board text removed: "PCB3D_BR_K40PositionalGuide"
- board text removed: "PCB3D_TL_K40PositionalGuide"
